File: Feather-NEO-M9N-GPS.sch (KiCad schematic (older format))
At the start: 50 parts, among them IC1 PRTR5V0U2F,115, J6 USB_B_Micro, U1 NEO-M9N, U2 AP2112K-3.3

Commit message: Rev2.1 of NEO-M9N
Parts:
- U1: footprint RF_GPS:ublox_NEO -> Feather-NEO-M9N-GPS:NEO-M9N
Changed lines of the file:
@@
 F 0 "U1" H 5500 4900 50  0000 C CNN
 F 1 "NEO-M9N" H 5500 4800 50  0000 C CNN
-F 2 "RF_GPS:ublox_NEO" H 5950 3100 50  0001 C CNN
+F 2 "Feather-NEO-M9N-GPS:NEO-M9N" H 5950 3100 50  0001 C CNN
 F 3 "https://www.u-blox.com/sites/default/files/NEO-M8-FW3_DataSheet_%28UBX-15031086%29.pdf" H 5550 3950 50  0001 C CNN
 	1    5550 3950

Commit message: Rev 2.2 designed
Lots of great feedback from the u-blox team. Hopefully this revision fixes a lot of the problems they pointed out
Parts:
- added JP13: MISO, Jumper:SolderJumper-2_P1.3mm_Open_RoundedPad1.0x1.5mm, symbol Jumper:SolderJumper_2_Open
- added JP14: MOSI, Jumper:SolderJumper-2_P1.3mm_Open_RoundedPad1.0x1.5mm, symbol Jumper:SolderJumper_2_Open
- added JP15: SCK, Jumper:SolderJumper-2_P1.3mm_Open_RoundedPad1.0x1.5mm, symbol Jumper:SolderJumper_2_Open
- added JP16: ~CS, Jumper:SolderJumper-2_P1.3mm_Open_RoundedPad1.0x1.5mm, symbol Jumper:SolderJumper_2_Open
- added R16, R17, R18, R19: 33, Resistor_SMD:R_0402_1005Metric, symbol Device:R_US
- JP4: value SPI1 -> SPI; footprint ~Jumper:SolderJumper-2_P1.3mm_Open_RoundedPad1.0x1.5mm -> Jumper:SolderJumper-2_P1.3mm_Open_RoundedPad1.0x1.5mm
- JP5: value ~RESET_GPS -> ~RST GPS
- R1, R2, R3, R4: footprint Resistor_SMD:R_0603_1608Metric -> Resistor_SMD:R_0402_1005Metric
- R13: value 1k -> 500
Connections:
- net 9`: now also JP16.1 (A)
- net INT: now also R17.1; no longer U1.4 (EXTINT)
- net MISO: now also J2.13 (Pin_13), JP13.1 (A)
- net MOSI: now also J2.12 (Pin_12), JP14.2 (B)
- net PPS: now also R18.1; no longer U1.3 (TIMEPULSE)
- net SCK: now also J2.11 (Pin_11), JP15.1 (A)
- net SCL: now also JP7.2 (B); no longer JP7.1 (A)
- net SDA: now also JP6.2 (B); no longer JP6.1 (A)
- net ~RESET_GPS: now also R16.1; no longer U1.8 (~RESET)
- net ~SAFE: now also R19.1; no longer U1.1 (~SAFEBOOT)
- net at R1.1: now also JP6.1 (A), JP16.2 (B); no longer JP6.2 (B)
- net at R2.1: now also JP7.1 (A), JP15.2 (B); no longer JP7.2 (B)
- net at JP8.1 (A), R3.1: now also JP14.1 (A)
- net at JP9.2 (B), R4.1: now also JP13.2 (B)
- new net: R19.2, U1.1 (~SAFEBOOT)
- new net: R18.2, U1.3 (TIMEPULSE)
- new net: R17.2, U1.4 (EXTINT)
- new net: R16.2, U1.8 (~RESET)
Other:
- note added: "Aspects not implemented\ndue to size restrictions"
- note added: "Choose which pin for digital I/O"
- note added: "Close to Enable SPI\nOpen enables UART, I2C"
- note removed: "Possible Pin Uses"
- note removed: "Though not used,\nClose to enable SPI"
- moved on the sheet: J4, J5, JP4, JP6, JP7, JP8, JP9, R14
