File: Feather-NEO-M9N-GPS.sch (KiCad schematic (older format))
At the start: 58 parts, among them IC1 PRTR5V0U2F,115, J6 USB_B_Micro, U1 NEO-M9N, U2 AP2112K-3.3

Commit message: Added additional CS pin. Kept caps as is because of integration manual
Parts:
- added JP17: ~CS2, Jumper:SolderJumper-2_P1.3mm_Open_RoundedPad1.0x1.5mm, symbol Jumper:SolderJumper_2_Open
Connections:
- net 6: now also JP17.1 (A)
- net at JP16.2 (B), JP6.1 (A), R1.1: now also JP17.2 (B)
Other:
- moved on the sheet: JP15, JP7
Changed lines of the file:
@@
 	10650 1650 10550 1650
-Wire Wire Line
-	10550 1550 10650 1550
 Wire Wire Line
 	10550 950  10650 950
@@
 Text Label 8150 4350 3    50   ~ 0
 TX
-Text Label 8350 3050 1    50   ~ 0
+Text Label 8700 3050 1    50   ~ 0
 SCL
 Text Label 7700 2950 1    50   ~ 0
@@
 L Jumper:SolderJumper_2_Bridged JP7
 U 1 1 5E2241A7
-P 8350 3300
-F 0 "JP7" H 8150 3400 50  0000 L CNN
-F 1 "SCL" H 8400 3400 50  0000 L CNN
-F 2 "Jumper:SolderJumper-2_P1.3mm_Bridged_RoundedPad1.0x1.5mm" H 8350 3300 50  0001 C CNN
-F 3 "~" H 8350 3300 50  0001 C CNN
-	1    8350 3300
+P 8700 3300
+F 0 "JP7" H 8500 3400 50  0000 L CNN
+F 1 "SCL" H 8750 3400 50  0000 L CNN
+F 2 "Jumper:SolderJumper-2_P1.3mm_Bridged_RoundedPad1.0x1.5mm" H 8700 3300 50  0001 C CNN
+F 3 "~" H 8700 3300 50  0001 C CNN
+	1    8700 3300
 	0    -1   -1   0
 $EndComp
@@
 	7700 3050 7700 2950
 Wire Wire Line
-	8350 3050 8350 3150
+	8700 3050 8700 3150
 $Comp
 L Jumper:SolderJumper_2_Open JP9
@@
 L Jumper:SolderJumper_2_Open JP15
 U 1 1 5E5C545C
-P 8600 3300
-F 0 "JP15" H 8700 3400 50  0000 L CNN
-F 1 "SCK" H 8400 3400 50  0000 L CNN
-F 2 "Jumper:SolderJumper-2_P1.3mm_Open_RoundedPad1.0x1.5mm" H 8600 3300 50  0001 C CNN
-F 3 "~" H 8600 3300 50  0001 C CNN
-	1    8600 3300
-	0    1    1    0
-$EndComp
-Wire Wire Line
-	8350 3550 8350 3450
-Wire Wire Line
-	6750 3550 8350 3550
-Wire Wire Line
-	8350 3550 8600 3550
-Wire Wire Line
-	8600 3550 8600 3450
-Connection ~ 8350 3550
-Text Label 8600 3050 1    50   ~ 0
+P 8950 3300
+F 0 "JP15" H 9050 3400 50  0000 L CNN
+F 1 "SCK" H 8750 3400 50  0000 L CNN
+F 2 "Jumper:SolderJumper-2_P1.3mm_Open_RoundedPad1.0x1.5mm" H 8950 3300 50  0001 C CNN
+F 3 "~" H 8950 3300 50  0001 C CNN
+	1    8950 3300
+	0    1    1    0
+$EndComp
+Wire Wire Line
+	8700 3550 8700 3450
+Wire Wire Line
+	8700 3550 8950 3550
+Wire Wire Line
+	8950 3550 8950 3450
+Connection ~ 8700 3550
+Text Label 8950 3050 1    50   ~ 0
 SCK
 Wire Wire Line
-	8600 3050 8600 3150
+	8950 3050 8950 3150
 Text Label 10050 1600 2    50   ~ 0
 ~CS
@@
 Wire Wire Line
 	10650 2300 10550 2300
+Wire Wire Line
+	6750 3550 8700 3550
+$Comp
+L Jumper:SolderJumper_2_Open JP17
+U 1 1 5E83C2E4
+P 8200 3200
+F 0 "JP17" H 8300 3300 50  0000 L CNN
+F 1 "~CS2" H 8000 3300 50  0000 L CNN
+F 2 "Jumper:SolderJumper-2_P1.3mm_Open_RoundedPad1.0x1.5mm" H 8200 3200 50  0001 C CNN
+F 3 "~" H 8200 3200 50  0001 C CNN
+	1    8200 3200
+	0    1    1    0
+$EndComp
+Wire Wire Line
+	8200 3350 8200 3450
+Wire Wire Line
+	8200 3450 7950 3450
+Connection ~ 7950 3450
+Text Label 8200 2950 1    50   ~ 0
+~CS2
+Wire Wire Line
+	8200 2950 8200 3050
+Text Label 10050 1700 2    50   ~ 0
+~CS2
+Wire Wire Line
+	10050 1700 10250 1700
+Wire Wire Line
+	10250 1700 10250 1550
+Wire Wire Line
+	10250 1550 10650 1550
 $EndSCHEMATC

Commit message: Updates
Parts:
- ANT1: symbol SamacSys_Parts:U.FL -> Feather-NEO-M9N-GPS-rescue:U.FL-SamacSys_Parts
- IC1: symbol SamacSys_Parts:PRTR5V0U2F,115 -> Feather-NEO-M9N-GPS-rescue:PRTR5V0U2F,115-SamacSys_Parts
- J6: symbol Connector:USB_B_Micro -> Feather-NEO-M9N-GPS-rescue:USB_B_Micro-Connector
- U1: symbol RF_GPS:u-blox_NEO-M9N -> Feather-NEO-M9N-GPS-rescue:u-blox_NEO-M9N-RF_GPS
- U2: symbol Regulator_Linear:AP2112K-3.3 -> Feather-NEO-M9N-GPS-rescue:AP2112K-3.3-Regulator_Linear
Changed lines of the file:
@@
 EESchema Schematic File Version 4
-LIBS:Feather-NEO-M9N-GPS-cache
 EELAYER 30 0
 EELAYER END
@@
 $EndComp
 $Comp
-L Connector:USB_B_Micro J6
+L Feather-NEO-M9N-GPS-rescue:USB_B_Micro-Connector J6
 U 1 1 5E0DB57B
 P 2850 1100
@@
 NoConn ~ 3150 1300
 $Comp
-L SamacSys_Parts:PRTR5V0U2F,115 IC1
+L Feather-NEO-M9N-GPS-rescue:PRTR5V0U2F,115-SamacSys_Parts IC1
 U 1 1 5E16E12C
 P 4300 1200
@@
 	6200 5650 6500 5650
 $Comp
-L Regulator_Linear:AP2112K-3.3 U2
+L Feather-NEO-M9N-GPS-rescue:AP2112K-3.3-Regulator_Linear U2
 U 1 1 5E148816
 P 6900 1200
@@
 Connection ~ 2500 3650
 $Comp
-L SamacSys_Parts:U.FL ANT1
+L Feather-NEO-M9N-GPS-rescue:U.FL-SamacSys_Parts ANT1
 U 1 1 5E064AD8
 P 1800 4500
@@
 $EndComp
 $Comp
-L RF_GPS:u-blox_NEO-M9N U1
+L Feather-NEO-M9N-GPS-rescue:u-blox_NEO-M9N-RF_GPS U1
 U 1 1 5E028BBB
 P 5550 3950
